Commit message: ...

File: dexopt/models/invisible_box.xacro (robot description, xacro)
@@ -6,22 +6,31 @@
     xmlns:xacro="http://playerstage.sourceforge.net/gazebo/xmlschema/#interface"
     name="simple_box">
+    <xacro:macro name="invisible_box_link" params="name sx sy sz mass">
+      <link name="${name}">
+          <inertial>
+              <mass value="${mass}"/>
+              <origin xyz="0 0 0" rpy="0 0 0"/>
+              <inertia
+                  ixx="${1.0/12*mass*(sy*sy+sz*sz)}" ixy="0" ixz="0"
+                  iyy="${1.0/12*mass*(sx*sx+sz*sz)}" iyz="0"
+                  izz="${1.0/12*mass*(sx*sx+sy*sy)}"
+                  />
+          </inertial>
+          <collision>
+              <origin xyz="0 0 0" rpy="0 0 0"/>
+              <geometry>
+                  <box size="${sx} ${sy} ${sz}"/>
+              </geometry>
+          </collision>
+      </link>
+    </xacro:macro>
     <xacro:macro name="invisible_box" params="name parent sx sy sz mass type:=fixed *origin">
-        <link name="${name}">
-            <inertial>
-                <mass value="${mass}"/>
-                <origin xyz="0 0 0" rpy="0 0 0"/>
-                <inertia
-                    ixx="${1.0/12*mass*(sy*sy+sz*sz)}" ixy="0" ixz="0"
-                    iyy="${1.0/12*mass*(sx*sx+sz*sz)}" iyz="0"
-                    izz="${1.0/12*mass*(sx*sx+sy*sy)}"
-                    />
-            </inertial>
-            <collision>
-                <origin xyz="0 0 0" rpy="0 0 0"/>
-                <geometry>
-                    <box size="${sx} ${sy} ${sz}"/>
-                </geometry>
-            </collision>
-        </link>
+        <xacro:invisible_box_link
+          name="${name}"
+          sx="${sx}"
+          sy="${sy}"
+          sz="${sz}"
+          mass="${mass}"
+          />
         <joint name="${name}_joint" type="${type}">
             <parent link="${parent}"/>

File: dexopt/worlds/grasp.xacro (robot description, xacro)
@@ -21,4 +21,7 @@
         wrist_1_upper_limit="${4.0*pi}"
         />
+    <xacro:include filename="$(find sr_description)/hand/xacro/full_hand.urdf.xacro"/>
+    <xacro:include filename="$(find sr_description)/other/xacro/gazebo/gazebo.urdf.xacro"/>
+    <xacro:shadowhand muscletrans="false" muscle="false" bio="false" bt_sp="false" ubi="false" eli="false" reflect="1.0" prefix="" lf="true"/>
     <joint name="world_arm_joint" type="fixed">
       <parent link="world" />
@@ -26,7 +29,13 @@
       <origin xyz="-0.75 -0.15 0" rpy="0 0 0" />
     </joint>
-    <xacro:include filename="$(find sr_description)/hand/xacro/full_hand.urdf.xacro"/>
-    <xacro:include filename="$(find sr_description)/other/xacro/gazebo/gazebo.urdf.xacro"/>
-    <xacro:shadowhand muscletrans="false" muscle="false" bio="false" bt_sp="false" ubi="false" eli="false" reflect="1.0" prefix="" lf="true"/>
+    <!--
+    <xacro:include filename="$(find tams_motorhand_description)/urdf/tams_motorhand.urdf.xacro"/>
+    <xacro:tams_motorhand type="left_pst" prefix="" />
+    <joint name="world_arm_joint" type="fixed">
+      <parent link="world" />
+      <child link="arm_base_link" />
+      <origin xyz="-0.75 -0.07 0" rpy="0 0 0" />
+    </joint>
+  -->
     <joint name="arm_hand_joint" type="fixed">
       <parent link="arm_ee_link" />
@@ -34,4 +43,11 @@
       <origin xyz="0.0 0.0 0.0" rpy="${pi/-2} 0 ${pi/-2}" />
     </joint>
+    <xacro:include filename="$(find dexopt)/objects/cube.xacro"/>
+    <joint name="object_joint" type="floating">
+      <parent link="world" />
+      <child link="object" />
+      <origin xyz="0 0 0.03" rpy="0 0 0"/>
+    </joint>
+    <!--
     <xacro:macro name="invisible_box" params="name parent sx sy sz mass type:=fixed *origin">
         <link name="${name}">
@@ -58,20 +74,5 @@
         </joint>
     </xacro:macro>
-    <xacro:invisible_box type="floating" name="object" parent="world" sx="0.06" sy="0.06" sz="0.06" mass="0.01">
-        <origin xyz="0 0 0.03" rpy="0 0 0"/>
-    </xacro:invisible_box>
-    <link name="object_visual">
-        <visual>
-            <geometry>
-                <mesh filename="package://dexopt/models/cube02.dae" scale="0.03 0.03 0.03"/>
-            </geometry>
-            <origin rpy="0 0 0" xyz="0 0 0"/>
-        </visual>
-    </link>
-    <joint name="object_visual_joint" type="fixed">
-      <parent link="object" />
-      <child link="object_visual" />
-      <origin xyz="0 0 0" rpy="0 0 0" />
-    </joint>
+    -->
     <xacro:invisible_box type="fixed" name="floor" parent="world" sx="0.5" sy="0.5" sz="0.4" mass="1">
         <origin xyz="0 0 -0.2" rpy="0 0 0"/>
