Commit message: .

File: dexopt/worlds/collision.xacro (robot description, xacro)
@@ -8,12 +8,12 @@
     <xacro:include filename="$(find dexopt)/models/simple_box.xacro"/>
     <link name="world"/>
-    <xacro:simple_box name="object" parent="world" sx="0.1" sy="0.1" sz="0.1" mass="1" type="floating">
+    <xacro:simple_box name="object" parent="world" sx="0.1" sy="0.1" sz="0.1" mass="1" type="floating" color="1 0 0 1">
       <origin xyz="0 0 0" rpy="0 0 0"/>
     </xacro:simple_box>
-    <xacro:simple_box name="object_2" parent="world" sx="0.5" sy="0.5" sz="0.5" mass="1">
-      <origin xyz="1 0 0" rpy="0 0 0"/>
+    <xacro:simple_box name="object_2" parent="world" sx="0.3" sy="0.3" sz="0.3" mass="1" color="0 1 0 1">
+      <origin xyz="-0.3 0 0" rpy="0 0 0"/>
     </xacro:simple_box>
-    <xacro:simple_box name="object_3" parent="world" sx="0.1" sy="0.1" sz="0.1" mass="1">
-      <origin xyz="0 1 0" rpy="0 0 0"/>
+    <xacro:simple_box name="object_3" parent="world" sx="0.1" sy="0.1" sz="0.1" mass="1" color="0 0 1 1">
+      <origin xyz="0 0.3 0" rpy="0 0 0"/>
     </xacro:simple_box>
 </robot>
