Commit message: turn, gazebo, ...

File: dexopt/worlds/turn.xacro (robot description, xacro)
@@ -14,5 +14,5 @@
       <parent link="world" />
       <child link="forearm" />
-      <origin xyz="0.0 0.30 0.24" rpy="${pi/2+pi/7} 0.0 0.0" />
+      <origin xyz="0.0 0.30 0.21" rpy="${pi/2+pi/10} 0.0 0.0" />
     </joint>
     <xacro:include filename="$(find dexopt)/objects/cylinder.xacro"/>
