Commit message: turn, ...

File: dexopt/objects/cube.xacro (robot description, xacro)
@@ -6,4 +6,31 @@
   xmlns:xacro="http://playerstage.sourceforge.net/gazebo/xmlschema/#interface"
   name="object">
+  <xacro:macro name="cube_object" params="name sx sy sz mass">
+    <link name="${name}">
+        <inertial>
+            <mass value="${mass}"/>
+            <origin xyz="0 0 0" rpy="0 0 0"/>
+            <inertia
+                ixx="${1.0/12*mass*(sy*sy+sz*sz)}" ixy="0" ixz="0"
+                iyy="${1.0/12*mass*(sx*sx+sz*sz)}" iyz="0"
+                izz="${1.0/12*mass*(sx*sx+sy*sy)}"
+                />
+        </inertial>
+        <collision>
+            <origin xyz="0 0 0" rpy="0 0 0"/>
+            <geometry>
+                <box size="${sx} ${sy} ${sz}"/>
+            </geometry>
+        </collision>
+        <visual>
+          <origin rpy="0 0 0" xyz="0 0 0"/>
+          <geometry>
+              <mesh filename="package://dexopt/models/cube02.dae" scale="${sx/2} ${sy/2} ${sz/2}"/>
+          </geometry>
+        </visual>
+    </link>
+  </xacro:macro>
+  <xacro:cube_object name="object" sx="0.06" sy="0.06" sz="0.06" mass="0.01"/>
+  <!--
   <xacro:include filename="$(find dexopt)/models/invisible_box.xacro"/>
   <xacro:invisible_box_link name="object" sx="0.06" sy="0.06" sz="0.06" mass="0.01"/>
@@ -21,3 +48,4 @@
     <origin xyz="0 0 0" rpy="0 0 0" />
   </joint>
+-->
 </robot>

File: dexopt/worlds/grasp2.xacro (robot description, xacro)
@@ -7,4 +7,5 @@
     xmlns:interface="http://playerstage.sourceforge.net/gazebo/xmlschema/#interface">
     <xacro:include filename="$(find dexopt)/models/simple_box.xacro"/>
+    <xacro:include filename="$(find dexopt)/models/invisible_box.xacro"/>
     <link name="world"/>
     <xacro:include filename="$(find sr_description)/hand/xacro/full_hand.urdf.xacro"/>

File: dexopt/worlds/grasp3.xacro (robot description, xacro)
@@ -7,12 +7,58 @@
     xmlns:interface="http://playerstage.sourceforge.net/gazebo/xmlschema/#interface">
     <xacro:include filename="$(find dexopt)/models/simple_box.xacro"/>
+    <xacro:include filename="$(find dexopt)/models/invisible_box.xacro"/>
     <link name="world"/>
     <xacro:include filename="$(find sr_description)/hand/xacro/full_hand.urdf.xacro"/>
     <xacro:include filename="$(find sr_description)/other/xacro/gazebo/gazebo.urdf.xacro"/>
     <xacro:shadowhand muscletrans="false" muscle="false" bio="false" bt_sp="false" ubi="false" eli="false" reflect="1.0" prefix="" lf="true"/>
+    <!--
     <joint name="world_hand_joint" type="floating">
       <parent link="world"/>
       <child link="forearm"/>
       <origin xyz="-0.35 -0.02 0.135" rpy="${pi/-2} ${pi} ${pi/-2}"/>
+    </joint>
+    -->
+    <link name="hand_x_link"/>
+    <joint name="hand_x" type="fixed">
+      <origin xyz="0 0 0" rpy="0 0 0"/>
+      <parent link="world"/>
+      <child link="hand_x_link"/>
+      <!--<axis xyz="1 0 0"/>
+      <limit effort="100" velocity="10" lower="0" upper="0.01"/>-->
+    </joint>
+    <link name="hand_y_link"/>
+    <joint name="hand_y" type="prismatic">
+      <origin xyz="0 0 0" rpy="0 0 0"/>
+      <parent link="hand_x_link"/>
+      <child link="hand_y_link"/>
+      <axis xyz="0 1 0"/>
+      <limit effort="100" velocity="10" lower="-0.01" upper="0.01"/>
+    </joint>
+    <link name="hand_z_link"/>
+    <joint name="hand_z" type="prismatic">
+      <origin xyz="0 0 0.06" rpy="0 0 0"/>
+      <parent link="hand_y_link"/>
+      <child link="hand_z_link"/>
+      <axis xyz="0 0 1"/>
+      <limit effort="100" velocity="10" lower="-0.2" upper="0.2"/>
+    </joint>
+    <link name="hand_pan_link"/>
+    <joint name="hand_pan" type="revolute">
+      <parent link="hand_z_link"/>
+      <child link="hand_pan_link"/>
+      <axis xyz="0 0 1"/>
+      <limit effort="100" velocity="10" lower="${pi*-0.1}" upper="${pi*0.1}"/>
+    </joint>
+    <link name="hand_tilt_link"/>
+    <joint name="hand_tilt" type="revolute">
+      <parent link="hand_pan_link"/>
+      <child link="hand_tilt_link"/>
+      <axis xyz="0 1 0"/>
+      <limit effort="100" velocity="10" lower="0" upper="${pi*0.1}"/>
+    </joint>
+    <joint name="world_hand_joint" type="fixed">
+      <parent link="hand_tilt_link"/>
+      <child link="forearm"/>
+      <origin xyz="-0.35 -0.02 0.075" rpy="${pi/-2} ${pi} ${pi/-2}"/>
     </joint>
     <xacro:include filename="$(find dexopt)/objects/cube.xacro"/>

File: dexopt/worlds/turn.xacro (robot description, xacro)
@@ -14,23 +14,16 @@
       <parent link="world" />
       <child link="forearm" />
-      <origin xyz="-0.01 0.30 0.24" rpy="${pi/2+pi/7} 0.0 0.0" />
+      <origin xyz="0.0 0.30 0.24" rpy="${pi/2+pi/7} 0.0 0.0" />
     </joint>
-    <xacro:invisible_cylinder type="floating" name="object" parent="world" radius="0.04" length="0.06" mass="0.1">
-        <origin xyz="0 0 0.025" rpy="0 0 0"/>
-    </xacro:invisible_cylinder>
-    <link name="object_visual">
-        <visual>
-            <geometry>
-                <mesh filename="package://dexopt/models/cylinder02.dae" scale="1 1 1"/>
-            </geometry>
-            <origin rpy="0 0 0" xyz="0 0 0"/>
-        </visual>
-    </link>
-    <joint name="object_visual_joint" type="fixed">
-      <parent link="object" />
-      <child link="object_visual" />
-      <origin xyz="0 0 0" rpy="0 0 0" />
+    <xacro:include filename="$(find dexopt)/objects/cylinder.xacro"/>
+    <joint name="object_joint" type="floating">
+      <parent link="world" />
+      <child link="object" />
+      <origin xyz="0 0 0.025" rpy="0 0 0"/>
     </joint>
-    <xacro:macro name="invisible_box" params="name parent sx sy sz mass type:=fixed *origin">
+    <xacro:simple_box type="fixed" name="floor" parent="world" sx="0.5" sy="0.5" sz="0.2" mass="1">
+        <origin xyz="0 0 -0.09" rpy="0 0 0"/>
+    </xacro:simple_box>
+    <!-- <xacro:macro name="invisible_box" params="name parent sx sy sz mass type:=fixed *origin">
         <link name="${name}">
             <inertial>
@@ -58,4 +51,4 @@
     <xacro:invisible_box type="fixed" name="floor" parent="world" sx="0.5" sy="0.5" sz="0.2" mass="1">
         <origin xyz="0 0 -0.1" rpy="0 0 0"/>
-    </xacro:invisible_box>
+    </xacro:invisible_box> -->
 </robot>
